Commit message: gazebo sim

File: robot_make/src/robot_description/urdf/mybot/base.urdf.xacro (robot description, xacro)
@@ -1,5 +1,7 @@
 <?xml version="1.0"?>
 <robot xmlns:xacro="http://www.ros.org/wiki/xacro">
+    <xacro:include filename="$(find robot_description)/urdf/mybot/common_inertial.xacro"/>
     <xacro:macro name="base_xacro" params="length radius">
+        <link name="base_footprint" />
         <link name="base_link">
             <visual>
@@ -12,5 +14,20 @@
                 </material>
             </visual>
+            <collision>
+                <origin xyz="0.0 0.0 0.0" rpy="0.0 0.0 0.0"/>
+                <geometry>
+                    <cylinder radius="${radius}" length="${length}"/>
+                </geometry>
+                <material name="white">
+                    <color rgba="1.0 1.0 1.0 0.5"/>
+                </material>
+            </collision>
+            <xacro:cylinder_inertia m="1.0" r="${radius}" h="${length}" />
         </link>
+        <joint name="joint_name" type="fixed">
+            <origin xyz="0.0 0.0 ${length/2.0+0.032-0.001}" rpy="0.0 0.0 0.0"/>
+            <parent link="base_footprint"/>
+            <child link="base_link"/>
+        </joint>
     </xacro:macro>
 </robot>

File: robot_make/src/robot_description/urdf/mybot/common_inertial.xacro (robot description, xacro)
@@ -18,6 +18,6 @@
         <inertial>
             <mass value="${m}"/>
-            <inertia ixx="${(2/5)*m*(r*r}" ixy="0.0" ixz="0.0" iyy="${(2/5)*m*(r*r}"
-                iyz="0.0" izz="${(2/5)*m*(r*r}"/>
+            <inertia ixx="${(2/5)*m*(r*r)}" ixy="0.0" ixz="0.0" iyy="${(2/5)*m*(r*r)}"
+                iyz="0.0" izz="${(2/5)*m*(r*r)}"/>
         </inertial>
     </xacro:macro>

File: robot_make/src/robot_description/urdf/mybot/mybot.urdf.xacro (robot description, xacro)
@@ -1,11 +1,23 @@
 <?xml version="1.0"?>
 <robot xmlns:xacro="http://www.ros.org/wiki/xacro" name="mybot">
+<!--主体部分库-->
 <xacro:include filename="$(find robot_description)/urdf/mybot/base.urdf.xacro"/>
+<!--传感器部分-->
 <xacro:include filename="$(find robot_description)/urdf/mybot/sensor/camera.urdf.xacro"/>
 <xacro:include filename="$(find robot_description)/urdf/mybot/sensor/imu.urdf.xacro"/>
 <xacro:include filename="$(find robot_description)/urdf/mybot/sensor/laser.urdf.xacro"/>
+<!--轮子部分-->
+<xacro:include filename="$(find robot_description)/urdf/mybot/actuator/wheel.urdf.xacro"/>
+<xacro:include filename="$(find robot_description)/urdf/mybot/actuator/caster.urdf.xacro"/>
+<!--主题声明-->
 <xacro:base_xacro length="0.12" radius="0.10" />
+<!--传感器-->
 <xacro:imu_xacro xyz="0.0 0.0 0.02" />
 <xacro:camera_xacro xyz="0.10 0.0 0.075" />
 <xacro:laser_xacro xyz="0.0 0.0 0.10" />
+<!--轮子-->
+<xacro:wheel_xacro wheel_name="left_wheel" xyz="0.0 0.10 -0.06" />
+<xacro:wheel_xacro wheel_name="right_wheel" xyz="0.0 -0.10 -0.06" />
+<xacro:caster_xacro caster_name="front_caster" xyz="0.08 0.0 -0.076" />
+<xacro:caster_xacro caster_name="back_caster" xyz="-0.08 0.0 -0.076" />
 </robot>

File: robot_make/src/robot_description/urdf/mybot/sensor/camera.urdf.xacro (robot description, xacro)
@@ -1,4 +1,5 @@
 <?xml version="1.0"?>
 <robot xmlns:xacro="http://www.ros.org/wiki/xacro">
+    <xacro:include filename="$(find robot_description)/urdf/mybot/common_inertial.xacro"/>
     <xacro:macro name="camera_xacro" params="xyz">
         <link name="camera_link">
@@ -12,4 +13,14 @@
                 </material>
             </visual>
+            <collision>
+                <origin xyz="0.0 0.0 0.0" rpy="0.0 0.0 0.0"/>
+                <geometry>
+                    <box size="0.02 0.10 0.02"/>
+                </geometry>
+                <material name="black">
+                    <color rgba="0.0 0.0 0.0 0.5"/>
+                </material>
+            </collision>
+            <xacro:cylinder_inertia m="0.05" r="0.01" h="0.02" />
         </link>
         <joint name="camera_joint" type="fixed">

File: robot_make/src/robot_description/urdf/mybot/sensor/imu.urdf.xacro (robot description, xacro)
@@ -1,4 +1,5 @@
 <?xml version="1.0"?>
 <robot xmlns:xacro="http://www.ros.org/wiki/xacro">
+    <xacro:include filename="$(find robot_description)/urdf/mybot/common_inertial.xacro"/>
     <xacro:macro name="imu_xacro" params="xyz">
         <link name="imu_link">
@@ -12,4 +13,14 @@
                 </material>
             </visual>
+            <collision>
+                <origin xyz="0.0 0.0 0.0" rpy="0.0 0.0 0.0"/>
+                <geometry>
+                    <box size="0.02 0.02 0.02"/>
+                </geometry>
+                <material name="black">
+                    <color rgba="0.0 0.0 0.0 0.5"/>
+                </material>
+            </collision>
+            <xacro:cylinder_inertia m="0.05" r="0.01" h="0.02" />
         </link>
         <joint name="imu_joint" type="fixed">

File: robot_make/src/robot_description/urdf/mybot/sensor/laser.urdf.xacro (robot description, xacro)
@@ -1,4 +1,5 @@
 <?xml version="1.0"?>
 <robot xmlns:xacro="http://www.ros.org/wiki/xacro">
+    <xacro:include filename="$(find robot_description)/urdf/mybot/common_inertial.xacro"/>
     <xacro:macro name="laser_xacro" params="xyz">
         <link name="laser_cylinder_link">
@@ -12,4 +13,14 @@
                 </material>
             </visual>
+            <collision>
+                <origin xyz="0.0 0.0 0.0" rpy="0.0 0.0 0.0"/>
+                <geometry>
+                    <cylinder radius="0.01" length="0.10"/>
+                </geometry>
+                <material name="black">
+                    <color rgba="0.0 0.0 0.0 1.0"/>
+                </material>
+            </collision>
+            <xacro:cylinder_inertia m="0.05" r="0.01" h="0.10" />
         </link>
         <link name="laser_link">
@@ -23,4 +34,14 @@
                 </material>
             </visual>
+            <collision>
+                <origin xyz="0.0 0.0 0.0" rpy="0.0 0.0 0.0"/>
+                <geometry>
+                    <cylinder radius="0.02" length="0.02"/>
+                </geometry>
+                <material name="black">
+                    <color rgba="0.0 0.0 0.0 1.0"/>
+                </material>
+            </collision>
+            <xacro:cylinder_inertia m="0.05" r="0.02" h="0.02" />
         </link>
         <joint name="laser_joint" type="fixed">
@@ -34,4 +55,10 @@
             <origin xyz="${xyz}" rpy="0.0 0.0 0.0"/>
         </joint>
+        <gazebo reference="laser_cylinder_joint">
+            <material>Gazebo/Black</material>
+        </gazebo>
+        <gazebo reference="laser_joint">
+            <material>Gazebo/Black</material>
+        </gazebo>
     </xacro:macro>
 </robot>
