Commit message: 1

File: robot_make/src/robot_description/urdf/mybot/sensor/camera.urdf.xacro (robot description, xacro)
@@ -3,12 +3,12 @@
     <xacro:include filename="$(find robot_description)/urdf/mybot/common_inertial.xacro"/>
     <xacro:macro name="camera_xacro" params="xyz">
-        <link name="camera_link">
+         <link name="camera_link">
             <visual>
-                <origin xyz="0.0 0.0 0.0" rpy="0.0 0.0 0.0"/>
+                <origin xyz="0 0 0.0" rpy="0 0 0" />
                 <geometry>
-                    <box size="0.02 0.10 0.02"/>
+                    <box size="0.02 0.10 0.02" />
                 </geometry>
                 <material name="black">
-                    <color rgba="0.0 0.0 0.0 0.5"/>
+                    <color rgba="0.0 0.0 0.0 0.8"/>
                 </material>
             </visual>
@@ -24,8 +24,14 @@
             <xacro:cylinder_inertia m="0.05" r="0.01" h="0.02" />
         </link>
+        <link name="camera_optical_link"></link>
+        <joint name="camera_optical_joint" type="fixed">
+            <parent link="camera_link" />
+            <child link="camera_optical_link" />
+            <origin xyz="0 0 0" rpy="${-pi/2} 0 ${-pi/2}" />
+        </joint>
         <joint name="camera_joint" type="fixed">
-            <parent link="base_link"/>
-            <child link="camera_link"/>
-            <origin xyz="${xyz}" rpy="0.0 0.0 0.0"/>
+            <parent link="base_link" />
+            <child link="camera_link" />
+            <origin xyz="${xyz}" />
         </joint>
     </xacro:macro>
